File: kicad/RD01/RD01_b.kicad_sch (KiCad schematic)
At the start: 8 parts

Commit message: 3
Parts:
- added Q?: 2N2219, Package_TO_SOT_THT:TO-39-3, symbol Transistor_BJT:2N2219
- added R?: 1K, symbol Device:R_Small
- added R?: 470, symbol Device:R_Small
Connections:
- net Earth: now also SW?.2, U?.-OUT (-SALIDA), U?.3 (GND), Q?.1 (E); no longer U?.4 (-out)
- net at U?.1 (+Vin): now also U?.+OUT (+SALIDA), R?.1; no longer SW?.2
- net at U?.2 (ctrl): now also SW?.1, Q?.3 (C), R?.2; no longer U?.-OUT (-SALIDA)
- net at Disp?.1 (VCC), Disp?.8 (LED), U?.1 (VCC)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: now also U?.4 (5V); no longer U?.3 (+out)
- net at U?.26 (GPIO_26): now also R?.1
- new net: Q?.2 (B), R?.2
Other:
- note added: "2N3904"
- note removed: "+5V"

Commit message: 10
Parts:
- removed Q?: 2N2219, Package_TO_SOT_THT:TO-39-3, symbol Transistor_BJT:2N2219
- removed U?: step_up, symbol Roberto:step_up
- added Q?: AO3400, Package_TO_SOT_SMD:SOT-23, symbol Transistor_FET:AO3400A
- added Q?: AO3401A, Package_TO_SOT_SMD:SOT-23, symbol Transistor_FET:AO3401A
- added R?: 51K, symbol Device:R_Small
- added R?: 68K, symbol Device:R_Small
- added R?: 10K, symbol Device:R_Small
- R?: value 1K -> 10K
- U?: value GM72 -> GM67 modificado
Connections:
- net Earth: now also Q?.2 (S), R?.1, R?.2
- net at R?.1: now also SW?.1, Q?.1 (G), Q?.3 (D); no longer U?.+OUT (+SALIDA)
- net at R?.2: now also U?.+OUT (+SALIDA), Q?.2 (S); no longer SW?.1
- net at Disp?.1 (VCC), Disp?.8 (LED), U?.BAT: now also Q?.3 (D), R?.2; no longer U?.1 (VCC)
- net at R?.2: now also Q?.1 (G), R?.1
- net at U?.35 (GPIO_35): now also R?.1, R?.2
- net at U?.3V (3V3): now also U?. (3.3V)
Other:
- note removed: "2N3904"

Commit message: 7
Parts:
- removed Q?: AO3400, Package_TO_SOT_SMD:SOT-23, symbol Transistor_FET:AO3400A
- removed Q?: AO3401A, Package_TO_SOT_SMD:SOT-23, symbol Transistor_FET:AO3401A
- removed R?: 51K, symbol Device:R_Small
- removed R?: 68K, symbol Device:R_Small
- removed R? (x2): 10K, symbol Device:R_Small
- removed R?: 470, symbol Device:R_Small
- added P1: esp 35, TestPoint:TestPoint_Pad_2.0x2.0mm, symbol Roberto:pad_2x2
- added P2: +Bat, TestPoint:TestPoint_Pad_2.0x2.0mm, symbol Roberto:pad_2x2
- added P3: esp 26, TestPoint:TestPoint_Pad_2.0x2.0mm, symbol Roberto:pad_2x2
- added P4: +Vcc, TestPoint:TestPoint_Pad_2.0x2.0mm, symbol Roberto:pad_2x2
- added P5: bot encend, TestPoint:TestPoint_Pad_2.0x2.0mm, symbol Roberto:pad_2x2
- added P6: GND, TestPoint:TestPoint_Pad_2.0x2.0mm, symbol Roberto:pad_2x2
- added Q1: AO3401, Package_TO_SOT_SMD:SOT-23, symbol Transistor_FET:AO3401A
- added Q2: AO3400, Package_TO_SOT_SMD:SOT-23, symbol Transistor_FET:AO3400A
- added R1: 51K, Resistor_THT:R_Axial_DIN0207_L6.3mm_D2.5mm_P10.16mm_Horizontal, symbol Device:R
- added R2: 470, Resistor_THT:R_Axial_DIN0207_L6.3mm_D2.5mm_P10.16mm_Horizontal, symbol Device:R
- added R3: 68K, Resistor_THT:R_Axial_DIN0207_L6.3mm_D2.5mm_P10.16mm_Horizontal, symbol Device:R
- added R4: 1K, Resistor_THT:R_Axial_DIN0207_L6.3mm_D2.5mm_P10.16mm_Horizontal, symbol Device:R
- added R5: 4K7, Resistor_THT:R_Axial_DIN0207_L6.3mm_D2.5mm_P10.16mm_Horizontal, symbol Device:R
Connections:
- net Earth: now also P6.1, Q2.2 (S), R3.2, R4.2
- net at SW?.1: now also P5.1, Q1.1 (G), Q2.3 (D), R5.1
- net at U?.+OUT (+SALIDA): now also P2.1, Q1.2 (S), R1.2, R5.2
- net at Disp?.1 (VCC), Disp?.8 (LED), U?.BAT: now also P4.1, Q1.3 (D)
- net at U?.26 (GPIO_26): now also P3.1, R2.1
- new net: Q2.1 (G), R2.2, R4.1
- new net: P1.1, R1.1, R3.1
