File: kicad/RD01/RD01_b.kicad_sch (KiCad schematic)
At the start: 20 parts, among them P1 esp 35, P2 +Bat, P3 esp 26, P4 +Vcc, P5 bot encend, P6 GND, Q1 AO3401, Q2 PN2222

Commit message: 10
Parts:
- Q1: value AO3401 -> DMG2305UX-7
Changed lines of the file:
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@@
   (junction (at 124.46 119.38) (diameter 0) (color 0 0 0 0)
   )
-  (junction (at 160.02 124.46) (diameter 0) (color 0 0 0 0)
+  (junction (at 161.29 124.46) (diameter 0) (color 0 0 0 0)
   )
   (wire (pts (xy 138.43 114.3) (xy 138.43 116.84))
     (stroke (width 0) (type default) (color 0 0 0 0))
   )
-  (wire (pts (xy 146.05 124.46) (xy 160.02 124.46))
+  (wire (pts (xy 146.05 124.46) (xy 161.29 124.46))
     (stroke (width 0) (type default) (color 0 0 0 0))
   )
@@
     (stroke (width 0) (type default) (color 0 0 0 0))
   )
-  (wire (pts (xy 160.02 93.98) (xy 160.02 124.46))
+  (wire (pts (xy 161.29 93.98) (xy 161.29 124.46))
     (stroke (width 0) (type default) (color 0 0 0 0))
   )
@@
     (stroke (width 0) (type default) (color 0 0 0 0))
   )
-  (wire (pts (xy 134.62 93.98) (xy 160.02 93.98))
+  (wire (pts (xy 134.62 93.98) (xy 161.29 93.98))
     (stroke (width 0) (type default) (color 0 0 0 0))
   )
@@
     (stroke (width 0) (type default) (color 0 0 0 0))
   )
-  (wire (pts (xy 160.02 124.46) (xy 165.1 124.46))
-    (stroke (width 0) (type default) (color 0 0 0 0))
-  )
   (wire (pts (xy 144.78 63.5) (xy 121.92 63.5))
     (stroke (width 0) (type default) (color 0 0 0 0))
   )
   (wire (pts (xy 124.46 55.88) (xy 121.92 55.88))
+    (stroke (width 0) (type default) (color 0 0 0 0))
+  )
+  (wire (pts (xy 161.29 124.46) (xy 165.1 124.46))
     (stroke (width 0) (type default) (color 0 0 0 0))
   )
@@
   )
   (symbol (lib_id "Transistor_FET:AO3401A") (at 143.51 114.3 0) (unit 1)
-    (in_bom yes) (on_board yes) (fields_autoplaced)
+    (in_bom yes) (on_board yes)
     (property "Reference" "Q1" (id 0) (at 149.86 113.0299 0)
       (effects (font (size 1.27 1.27)) (justify left))
     )
-    (property "Value" "AO3401" (id 1) (at 149.86 115.5699 0)
+    (property "Value" "DMG2305UX-7" (id 1) (at 146.05 110.49 0)
       (effects (font (size 1.27 1.27)) (justify left))
     )
@@
     )
     (path "/4140cca9-a87f-4419-adc0-ee979fee5023"
-      (reference "Q1") (unit 1) (value "AO3401") (footprint "Package_TO_SOT_SMD:SOT-23")
+      (reference "Q1") (unit 1) (value "DMG2305UX-7") (footprint "Package_TO_SOT_SMD:SOT-23")
     )
     (path "/ca741e03-89b1-494a-bae9-b2cc6b3c072d"
