File: kicad/RD01/RD01_2/RD01_2.kicad_sch (KiCad schematic)
At the start: 13 parts, among them P1 +Vcc, P2 esp 26, P3 +Bat, P4 esp 35, P5 GND, Q1 DMG2305UX-7, Q2 PN2222A, SW1 encendido

Commit message: 10
Parts:
- removed Q1: DMG2305UX-7, Package_TO_SOT_SMD:SOT-23, symbol Transistor_FET:DMG2301L
- removed Q2: PN2222A, Package_TO_SOT_SMD:SOT-23, symbol Transistor_BJT:PN2222A
- added Q1: PN2222Asmd, Package_TO_SOT_SMD:SOT-23, symbol Transistor_BJT:PN2222A
- added Q2: DMG2305UX-7, Package_TO_SOT_SMD:SOT-23, symbol Transistor_FET:DMG2301L
- P1: value +Vcc -> esp 26
- P2: value esp 26 -> GND
- P3: value +Bat -> +Vcc
- P4: value esp 35 -> +Bat
- P5: value GND -> esp 35
- R1: value 10K -> 470
- R3: value 470 -> 68K
- R4: value 51K -> 10K
- R5: value 68K -> 51K
Connections:
- net at P4.1, R4.2: now also R5.1, Q2.2 (S); no longer R5.2
- net at R2.1: now also R1.2, Q1.1 (B); no longer R3.2
- net at R2.2, SW1.1: now also P2.1, R3.1, Q1.2 (E); no longer P5.1, R5.1
- net at SW1.2: now also R4.1, Q1.3 (C), Q2.1 (G); no longer R1.1
- net at P1.1: now also R1.1
- new net: P3.1, Q2.3 (D)
- new net: P5.1, R3.2, R5.2
