File: kicad/RD01/RD01_2/RD01_2_completo.kicad_sch (KiCad schematic)
At the start: 19 parts, among them P1 +Vcc, P2 esp 26, P3 +Bat, P4 esp 35, P5 GND, Q1 DMG2305UX-7, Q2 PN2222A, SW1 encendido

Commit message: 10
Parts:
- added P1: esp 35, TestPoint:TestPoint_Pad_2.0x2.0mm, symbol Roberto:pad_2x2
- added P2: +Bat, TestPoint:TestPoint_Pad_2.0x2.0mm, symbol Roberto:pad_2x2
- added P3: esp 26, TestPoint:TestPoint_Pad_2.0x2.0mm, symbol Roberto:pad_2x2
- added P4: +Vcc, TestPoint:TestPoint_Pad_2.0x2.0mm, symbol Roberto:pad_2x2
- added P5: bot encend, TestPoint:TestPoint_Pad_2.0x2.0mm, symbol Roberto:pad_2x2
- added P6: GND, TestPoint:TestPoint_Pad_2.0x2.0mm, symbol Roberto:pad_2x2
- added Q1: DMG2305UX-7, Package_TO_SOT_SMD:SOT-23, symbol Transistor_FET:AO3401A
- added Q2: PN2222, Package_TO_SOT_THT:TO-92_Inline, symbol Transistor_BJT:PN2222A
- added R1: 51K, Resistor_THT:R_Axial_DIN0207_L6.3mm_D2.5mm_P10.16mm_Horizontal, symbol Device:R
- added R2: 470, Resistor_THT:R_Axial_DIN0207_L6.3mm_D2.5mm_P10.16mm_Horizontal, symbol Device:R
- added R3: 68K, Resistor_THT:R_Axial_DIN0207_L6.3mm_D2.5mm_P10.16mm_Horizontal, symbol Device:R
- added R4, R5: 10K, Resistor_THT:R_Axial_DIN0207_L6.3mm_D2.5mm_P10.16mm_Horizontal, symbol Device:R
- added SW?: encendido, symbol Switch:SW_Push
Connections:
- net Earth: now also P6.1, Q2.1 (E), R3.2, R4.2, SW?.2; no longer P5.1, Q2.1 (E), R2.2, R5.1, SW1.1
- net at P3.1, Q1.2 (S), R1.2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: no longer U?.+OUT (+SALIDA)
- net at P4.1, R4.2, R5.2: no longer U?.35 (GPIO_35)
- net at Disp?.1 (VCC), Disp?.8 (LED), U?.BAT: now also P4.1, Q1.3 (D); no longer P1.1, Q1.3 (D)
- net at P2.1, R3.1: no longer U?.26 (GPIO_26)
- new net: P5.1, Q2.1 (E), R2.2, R5.1, SW1.1
- new net: P2.1, Q1.2 (S), R1.2, R5.2, U?.+OUT (+SALIDA)
- new net: P5.1, Q1.1 (G), Q2.3 (C), R5.1, SW?.1
- new net: P1.1, Q1.3 (D)
- new net: P3.1, R2.1, U?.26 (GPIO_26)
- new net: Q2.2 (B), R2.2, R4.1
- new net: P1.1, R1.1, R3.1
Other:
- moved on the sheet: P1, P2, P3, P4, P5, Q1, Q2, R1, R2, R3, R4, R5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
