File: circuito_impreso/RD01/RD01_b.kicad_sch (KiCad schematic)
At the start: 19 parts, among them P1 +Vcc, P2 esp 26, P3 +Bat, P4 esp 35, P5 GND, Q1 DMG2305UX-7, Q2 PN2222A, SW1 encendido

Commit message: 12
Parts:
- Q1: renamed from Q2; value PN2222A -> PN2222A smd
- renumbered P2 to P1, P5 to P2, P1 to P3, P3 to P4, P4 to P5, Q1 to Q2, R3 to R1, R5 to R3, R1 to R4, R4 to R5
Changed lines of the file:
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@@
   (symbol (lib_name "pad_2x2_4") (lib_id "Roberto:pad_2x2") (at 104.14 114.3 180) (unit 1)
     (in_bom yes) (on_board yes)
-    (property "Reference" "P5" (id 0) (at 105.41 118.11 0))
+    (property "Reference" "P2" (id 0) (at 105.41 118.11 0))
     (property "Value" "GND" (id 1) (at 105.41 111.76 0))
     (property "Footprint" "TestPoint:TestPoint_Pad_2.0x2.0mm" (id 2) (at 104.14 114.3 0)
@@
   (symbol (lib_id "Device:R") (at 153.67 118.11 0) (unit 1)
     (in_bom yes) (on_board yes)
-    (property "Reference" "R4" (id 0) (at 154.94 116.84 0)
+    (property "Reference" "R5" (id 0) (at 154.94 116.84 0)
       (effects (font (size 1.27 1.27)) (justify left))
     )
@@
   (symbol (lib_id "Transistor_BJT:PN2222A") (at 128.27 105.41 0) (unit 1)
     (in_bom yes) (on_board yes)
-    (property "Reference" "Q2" (id 0) (at 123.19 102.87 0)
-      (effects (font (size 1.27 1.27)) (justify left))
-    )
-    (property "Value" "PN2222A" (id 1) (at 120.65 100.33 0)
+    (property "Reference" "Q1" (id 0) (at 123.19 102.87 0)
+      (effects (font (size 1.27 1.27)) (justify left))
+    )
+    (property "Value" "PN2222A smd" (id 1) (at 118.11 99.06 0)
       (effects (font (size 1.27 1.27)) (justify left))
     )
@@
   (symbol (lib_name "pad_2x2_1") (lib_id "Roberto:pad_2x2") (at 162.56 113.03 0) (unit 1)
     (in_bom yes) (on_board yes)
-    (property "Reference" "P3" (id 0) (at 160.02 109.22 0)
+    (property "Reference" "P4" (id 0) (at 160.02 109.22 0)
       (effects (font (size 1.27 1.27)) (justify left))
     )
@@
   (symbol (lib_name "pad_2x2_2") (lib_id "Roberto:pad_2x2") (at 162.56 92.71 0) (unit 1)
     (in_bom yes) (on_board yes)
-    (property "Reference" "P1" (id 0) (at 160.02 93.98 0)
+    (property "Reference" "P3" (id 0) (at 160.02 93.98 0)
       (effects (font (size 1.27 1.27)) (justify left))
     )
@@
   (symbol (lib_id "Transistor_FET:DMG2301L") (at 154.94 100.33 0) (unit 1)
     (in_bom yes) (on_board yes)
-    (property "Reference" "Q1" (id 0) (at 146.05 93.98 0)
+    (property "Reference" "Q2" (id 0) (at 146.05 93.98 0)
       (effects (font (size 1.27 1.27)) (justify left))
     )
@@
   (symbol (lib_name "pad_2x2_5") (lib_id "Roberto:pad_2x2") (at 104.14 104.14 180) (unit 1)
     (in_bom yes) (on_board yes)
-    (property "Reference" "P2" (id 0) (at 105.41 107.95 0))
+    (property "Reference" "P1" (id 0) (at 105.41 107.95 0))
     (property "Value" "esp 26" (id 1) (at 105.41 101.6 0))
     (property "Footprint" "TestPoint:TestPoint_Pad_2.0x2.0mm" (id 2) (at 104.14 104.14 0)
@@
   (symbol (lib_id "Device:R") (at 149.86 107.95 0) (unit 1)
     (in_bom yes) (on_board yes)
-    (property "Reference" "R1" (id 0) (at 151.13 106.68 0)
+    (property "Reference" "R4" (id 0) (at 151.13 106.68 0)
       (effects (font (size 1.27 1.27)) (justify left))
     )
@@
   (symbol (lib_id "Device:R") (at 146.05 118.11 0) (unit 1)
     (in_bom yes) (on_board yes)
-    (property "Reference" "R5" (id 0) (at 147.32 116.84 0)
+    (property "Reference" "R3" (id 0) (at 147.32 116.84 0)
       (effects (font (size 1.27 1.27)) (justify left))
     )
@@
   (symbol (lib_id "Device:R") (at 115.57 105.41 90) (unit 1)
     (in_bom yes) (on_board yes)
-    (property "Reference" "R3" (id 0) (at 114.3 104.14 0)
+    (property "Reference" "R1" (id 0) (at 114.3 104.14 0)
       (effects (font (size 1.27 1.27)) (justify left))
     )
@@
   (symbol (lib_name "pad_2x2_3") (lib_id "Roberto:pad_2x2") (at 162.56 123.19 0) (unit 1)
     (in_bom yes) (on_board yes)
-    (property "Reference" "P4" (id 0) (at 161.29 119.38 0))
+    (property "Reference" "P5" (id 0) (at 161.29 119.38 0))
     (property "Value" "esp 35" (id 1) (at 161.29 125.73 0))
     (property "Footprint" "TestPoint:TestPoint_Pad_2.0x2.0mm" (id 2) (at 162.56 123.19 0)
@@
       (reference "J?") (unit 1) (value "Conn_Coaxial") (footprint "")
     )
+    (path "/bb08f64b-170a-47af-9dd4-18b48237a9ca"
+      (reference "P1") (unit 1) (value "esp 26") (footprint "TestPoint:TestPoint_Pad_2.0x2.0mm")
+    )
+    (path "/01467dd4-fd8c-4c9b-883f-656921ce0c2b"
+      (reference "P2") (unit 1) (value "GND") (footprint "TestPoint:TestPoint_Pad_2.0x2.0mm")
+    )
     (path "/3d0c0a89-1c30-42d8-8a26-0434997c3098"
-      (reference "P1") (unit 1) (value "+Vcc") (footprint "TestPoint:TestPoint_Pad_2.0x2.0mm")
-    )
-    (path "/bb08f64b-170a-47af-9dd4-18b48237a9ca"
-      (reference "P2") (unit 1) (value "esp 26") (footprint "TestPoint:TestPoint_Pad_2.0x2.0mm")
+      (reference "P3") (unit 1) (value "+Vcc") (footprint "TestPoint:TestPoint_Pad_2.0x2.0mm")
     )
     (path "/3bd0ecca-cabe-4dd9-8218-846b8fe47db2"
-      (reference "P3") (unit 1) (value "+Bat") (footprint "TestPoint:TestPoint_Pad_2.0x2.0mm")
+      (reference "P4") (unit 1) (value "+Bat") (footprint "TestPoint:TestPoint_Pad_2.0x2.0mm")
     )
     (path "/f7bd3697-37ec-4a3d-a807-621fb743c832"
-      (reference "P4") (unit 1) (value "esp 35") (footprint "TestPoint:TestPoint_Pad_2.0x2.0mm")
-    )
-    (path "/01467dd4-fd8c-4c9b-883f-656921ce0c2b"
-      (reference "P5") (unit 1) (value "GND") (footprint "TestPoint:TestPoint_Pad_2.0x2.0mm")
+      (reference "P5") (unit 1) (value "esp 35") (footprint "TestPoint:TestPoint_Pad_2.0x2.0mm")
+    )
+    (path "/270cac3c-8235-41d3-b167-c04a1079deef"
+      (reference "Q1") (unit 1) (value "PN2222A smd") (footprint "Package_TO_SOT_SMD:SOT-23")
     )
     (path "/5acbf5b2-38cf-41ed-aa3a-502d11b5411a"
-      (reference "Q1") (unit 1) (value "DMG2305UX-7") (footprint "Package_TO_SOT_SMD:SOT-23")
-    )
-    (path "/270cac3c-8235-41d3-b167-c04a1079deef"
-      (reference "Q2") (unit 1) (value "PN2222A") (footprint "Package_TO_SOT_SMD:SOT-23")
-    )
-    (path "/bb0e98e0-0635-413f-94f2-3b92ef733e45"
-      (reference "R1") (unit 1) (value "10K") (footprint "Resistor_SMD:R_1206_3216Metric_Pad1.30x1.75mm_HandSolder")
+      (reference "Q2") (unit 1) (value "DMG2305UX-7") (footprint "Package_TO_SOT_SMD:SOT-23")
+    )
+    (path "/d75fc856-cfcf-43a6-a339-d3cc663b5ecc"
+      (reference "R1") (unit 1) (value "470") (footprint "Resistor_SMD:R_1206_3216Metric_Pad1.30x1.75mm_HandSolder")
     )
     (path "/e5de7ad2-794e-4c22-88b8-2e720aabf58f"
       (reference "R2") (unit 1) (value "10K") (footprint "Resistor_SMD:R_1206_3216Metric_Pad1.30x1.75mm_HandSolder")
     )
-    (path "/d75fc856-cfcf-43a6-a339-d3cc663b5ecc"
-      (reference "R3") (unit 1) (value "470") (footprint "Resistor_SMD:R_1206_3216Metric_Pad1.30x1.75mm_HandSolder")
+    (path "/d71dd076-40a6-4ca9-a3bc-a90f30ba81de"
+      (reference "R3") (unit 1) (value "68K") (footprint "Resistor_SMD:R_1206_3216Metric_Pad1.30x1.75mm_HandSolder")
+    )
+    (path "/bb0e98e0-0635-413f-94f2-3b92ef733e45"
+      (reference "R4") (unit 1) (value "10K") (footprint "Resistor_SMD:R_1206_3216Metric_Pad1.30x1.75mm_HandSolder")
     )
     (path "/1bfbeba1-c13a-4984-8eaa-9e0e12769fd6"
-      (reference "R4") (unit 1) (value "51K") (footprint "Resistor_SMD:R_1206_3216Metric_Pad1.30x1.75mm_HandSolder")
-    )
-    (path "/d71dd076-40a6-4ca9-a3bc-a90f30ba81de"
-      (reference "R5") (unit 1) (value "68K") (footprint "Resistor_SMD:R_1206_3216Metric_Pad1.30x1.75mm_HandSolder")
+      (reference "R5") (unit 1) (value "51K") (footprint "Resistor_SMD:R_1206_3216Metric_Pad1.30x1.75mm_HandSolder")
     )
     (path "/902003f4-d94e-4465-a11e-7cac1aa1b9de"
